File: Placa_YM2612.sch (KiCad schematic (older format))
At the start: 24 parts, among them J1 Conn_02x18_Odd_Even, J2 Conn_01x02, J3 AudioJack3, U1 YM2612, U2 74LS74, U3 SN76489, U4 TL072, X1 8 MHz

Commit message: Placa a fabricar
Parts:
- removed U4: TL072, Package_DIP:DIP-8_W7.62mm_LongPads, symbol Amplifier_Operational:TL072
- added C6: 0.1u, Capacitor_THT:C_Disc_D5.0mm_W2.5mm_P2.50mm, symbol Device:C
- added U4: LM358, Package_DIP:DIP-8_W7.62mm_LongPads, symbol Amplifier_Operational:LM358
- U2: footprint (none) -> Package_DIP:DIP-14_W7.62mm_LongPads
Connections:
- net +5V: now also C6.1, U4.8 (V+)
- net GND: now also C6.2, U4.4 (V-)
- net at R3.1, R6.1, R8.2: now also U4.6 (-)
- net at R4.1, R7.1, R9.2: now also U4.2 (-)
- net at C5.1, R9.1: now also U4.1
- net at R10.2, R11.1: now also U4.3 (+), U4.5 (+)
- net at C4.1, R8.1: now also U4.7
Changed lines of the file:
@@
 	0    1    1    0
-$EndComp
-$Comp
-L Amplifier_Operational:TL072 U4
-U 1 1 5D34A540
-P 9250 2950
-F 0 "U4" H 9250 2583 50  0000 C CNN
-F 1 "TL072" H 9250 2674 50  0000 C CNN
-F 2 "Package_DIP:DIP-8_W7.62mm_LongPads" H 9250 2950 50  0001 C CNN
-F 3 "http://www.ti.com/lit/ds/symlink/tl071.pdf" H 9250 2950 50  0001 C CNN
-	1    9250 2950
-	1    0    0    1
 $EndComp
 Wire Wire Line
@@
 Wire Wire Line
 	8600 1850 8950 1850
-$Comp
-L Amplifier_Operational:TL072 U4
-U 2 1 5D3611C4
-P 9250 1950
-F 0 "U4" H 9250 1583 50  0000 C CNN
-F 1 "TL072" H 9250 1674 50  0000 C CNN
-F 2 "Package_DIP:DIP-8_W7.62mm_LongPads" H 9250 1950 50  0001 C CNN
-F 3 "http://www.ti.com/lit/ds/symlink/tl071.pdf" H 9250 1950 50  0001 C CNN
-	2    9250 1950
-	1    0    0    1
-$EndComp
 $Comp
 L Device:R_US R6
@@
 	10050 2400 10050 2200
 $Comp
-L Amplifier_Operational:TL072 U4
-U 3 1 5D40B140
-P 9750 3950
-F 0 "U4" H 9708 3996 50  0000 L CNN
-F 1 "TL072" H 9708 3905 50  0000 L CNN
-F 2 "Package_DIP:DIP-8_W7.62mm_LongPads" H 9750 3950 50  0001 C CNN
-F 3 "http://www.ti.com/lit/ds/symlink/tl071.pdf" H 9750 3950 50  0001 C CNN
-	3    9750 3950
-	1    0    0    -1
-$EndComp
-$Comp
 L power:GND #PWR019
 U 1 1 5D40E6C5
@@
 F 0 "U2" H 6930 5646 50  0000 L CNN
 F 1 "74LS74" H 6930 5555 50  0000 L CNN
-F 2 "" H 6700 5600 50  0001 C CNN
+F 2 "Package_DIP:DIP-14_W7.62mm_LongPads" H 6700 5600 50  0001 C CNN
 F 3 "74xx/74hc_hct74.pdf" H 6700 5600 50  0001 C CNN
 	3    6700 5600
@@
 Wire Wire Line
 	6700 5150 6700 5200
+$Comp
+L Device:C C6
+U 1 1 5D330663
+P 10150 3850
+F 0 "C6" H 10265 3896 50  0000 L CNN
+F 1 "0.1u" H 10265 3805 50  0000 L CNN
+F 2 "Capacitor_THT:C_Disc_D5.0mm_W2.5mm_P2.50mm" H 10188 3700 50  0001 C CNN
+F 3 "~" H 10150 3850 50  0001 C CNN
+	1    10150 3850
+	1    0    0    -1
+$EndComp
+Wire Wire Line
+	10150 3700 10150 3650
+Wire Wire Line
+	10150 3650 9650 3650
+$Comp
+L power:GND #PWR0101
+U 1 1 5D337545
+P 10150 4050
+F 0 "#PWR0101" H 10150 3800 50  0001 C CNN
+F 1 "GND" H 10155 3877 50  0000 C CNN
+F 2 "" H 10150 4050 50  0001 C CNN
+F 3 "" H 10150 4050 50  0001 C CNN
+	1    10150 4050
+	1    0    0    -1
+$EndComp
+Wire Wire Line
+	10150 4050 10150 4000
+$Comp
+L Amplifier_Operational:LM358 U4
+U 2 1 5D37BF72
+P 9250 1950
+F 0 "U4" H 9250 1583 50  0000 C CNN
+F 1 "LM358" H 9250 1674 50  0000 C CNN
+F 2 "Package_DIP:DIP-8_W7.62mm_LongPads" H 9250 1950 50  0001 C CNN
+F 3 "http://www.ti.com/lit/ds/symlink/lm2904-n.pdf" H 9250 1950 50  0001 C CNN
+	2    9250 1950
+	1    0    0    1
+$EndComp
+$Comp
+L Amplifier_Operational:LM358 U4
+U 1 1 5D385DB1
+P 9250 2950
+F 0 "U4" H 9250 2583 50  0000 C CNN
+F 1 "LM358" H 9250 2674 50  0000 C CNN
+F 2 "Package_DIP:DIP-8_W7.62mm_LongPads" H 9250 2950 50  0001 C CNN
+F 3 "http://www.ti.com/lit/ds/symlink/lm2904-n.pdf" H 9250 2950 50  0001 C CNN
+	1    9250 2950
+	1    0    0    1
+$EndComp
 Wire Bus Line
 	3100 2750 3100 4700
@@
 Wire Bus Line
 	2450 3050 2450 4700
+$Comp
+L Amplifier_Operational:LM358 U4
+U 3 1 5D390B5C
+P 9750 3950
+F 0 "U4" H 9708 3996 50  0000 L CNN
+F 1 "LM358" H 9708 3905 50  0000 L CNN
+F 2 "Package_DIP:DIP-8_W7.62mm_LongPads" H 9750 3950 50  0001 C CNN
+F 3 "http://www.ti.com/lit/ds/symlink/lm2904-n.pdf" H 9750 3950 50  0001 C CNN
+	3    9750 3950
+	1    0    0    -1
+$EndComp
+Connection ~ 9650 3650
 $EndSCHEMATC

Commit message: Corregidos nombres de los canales
Connections:
- net AUDIO_L: now also C5.2, J3.T; no longer C4.2, J3.R
- net AUDIO_R: now also C4.2, J3.R; no longer C5.2, J3.T
- net YM_LEFT: now also C2.1, R2.1, U1.21 (MOL); no longer C1.1, R1.1, U1.20 (MOR)
- net YM_RIGHT: now also C1.1, R1.1, U1.20 (MOR); no longer C2.1, R2.1, U1.21 (MOL)
Changed lines of the file:
@@
 EESchema Schematic File Version 4
 LIBS:Placa_YM2612-cache
-EELAYER 29 0
+EELAYER 30 0
 EELAYER END
 $Descr A4 11693 8268
@@
 Wire Wire Line
 	10050 2200 10400 2200
-Text Label 5250 2150 0    50   ~ 0
+Text Label 5700 2200 3    50   ~ 0
 YM_LEFT
-Text Label 5700 2200 3    50   ~ 0
+Text Label 5700 2150 2    50   ~ 0
 YM_RIGHT
 Text Label 7150 2850 0    50   ~ 0
 PSG_OUT
+Text Label 10050 2200 0    50   ~ 0
+AUDIO_L
 Text Label 10050 2100 0    50   ~ 0
-AUDIO_L
-Text Label 10050 2200 0    50   ~ 0
 AUDIO_R
 $Comp
@@
 	1    0    0    1
 $EndComp
-Wire Bus Line
-	3100 2750 3100 4700
-Wire Bus Line
-	5500 2750 5500 4700
-Wire Bus Line
-	2450 3050 2450 4700
 $Comp
 L Amplifier_Operational:LM358 U4
@@
 $EndComp
 Connection ~ 9650 3650
+Wire Bus Line
+	3100 2750 3100 4700
+Wire Bus Line
+	5500 2750 5500 4700
+Wire Bus Line
+	2450 3050 2450 4700
 $EndSCHEMATC
