File: Placa_YM2612.kicad_pcb (KiCad board)
At the start: 2 copper layers, 90.2 x 54.6 mm, 24 parts, among them J1 Conn_02x18_Odd_Even, J2 Conn_01x02, J3 AudioJack3, U1 YM2612, U2 74LS74, U3 SN76489, U4 TL072, X1 8 MHz

Commit message: Placa a fabricar
Parts:
- added C6: 0.1u, Capacitor_THT:C_Disc_D5.0mm_W2.5mm_P2.50mm, F.Cu at (142.2, 45.7)
- U4: value TL072 -> LM358
- moved U3 51.6 mm to (73.7, 86.4), turned to 90 degrees
- moved X1 41.6 mm to (114.3, 66.0), turned to 180 degrees
- moved R1 16.5 mm to (114.3, 55.9), turned to 90 degrees
- moved U2 15.9 mm to (97.8, 86.4), turned to 90 degrees
- moved U1 14.5 mm to (73.7, 59.7), turned to 90 degrees
- moved R2 11.7 mm to (109.2, 55.9)
- moved R8 10.2 mm to (144.8, 40.6), turned to 180 degrees
- moved R10 1.27 mm to (146.1, 45.7)
- moved C1 1.27 mm to (121.9, 66.0)
- moved C2 1.27 mm to (121.9, 73.7)
- moved C3 1.27 mm to (121.9, 82.5)
Routing:
- net /D3: track 154.2 -> 47.7 mm, vias 4 -> 2
- net /D2: track 146.7 -> 40.4 mm, vias 3 -> 2
- net /D1: track 145.3 -> 46.8 mm, vias 3 -> 2
- net /D0: track 127.9 -> 44.1 mm
- net /D5: track 143.0 -> 73.9 mm, vias 4 -> 0
- net /D4: track 120.2 -> 54.2 mm, vias 4 -> 2
- net /D6: track 132.0 -> 70.5 mm, vias 4 -> 0
- net GND: track 48.1 -> 0.00 mm, vias 10 -> 0
- net +5V: track 236.8 -> 198.7 mm, vias 7 -> 6
- net /CLK8: track 84.0 -> 116.5 mm, vias 5 -> 4
- net /YM_RIGHT: track 51.8 -> 79.1 mm, vias 4 -> 2
- net /YM_LEFT: track 41.7 -> 64.7 mm
- net /YM_A1: track 44.8 -> 25.9 mm
- net /YM_A0: track 43.9 -> 26.6 mm
- net /~YM_IC: track 53.1 -> 35.9 mm, vias 2 -> 0
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- removed copper zone on F.Cu, net GND

Commit message: Corregidos nombres de los canales
Connections:
- C1 pad 1: /YM_LEFT -> /YM_RIGHT
- C2 pad 1: /YM_RIGHT -> /YM_LEFT
- C4 pad 2: /AUDIO_L -> /AUDIO_R
- C5 pad 2: /AUDIO_R -> /AUDIO_L
- J3 pad R: /AUDIO_L -> /AUDIO_R
- J3 pad T: /AUDIO_R -> /AUDIO_L
- R1 pad 1: /YM_LEFT -> /YM_RIGHT
- R2 pad 1: /YM_RIGHT -> /YM_LEFT
- U1 pad 20: /YM_LEFT -> /YM_RIGHT
- U1 pad 21: /YM_RIGHT -> /YM_LEFT
Routing:
- net /YM_RIGHT: track 79.1 -> 64.7 mm
- net /YM_LEFT: track 64.7 -> 79.1 mm
- net /AUDIO_R: track 16.5 -> 23.9 mm
- net /AUDIO_L: track 23.9 -> 16.5 mm

Commit message: Inicio de modificaciones para enviar a PCBWay
Parts:
- moved J1 133.6 mm to (198.1, 53.3)
- moved R11 110.4 mm to (40.7, 72.4), turned to 0 degrees
- moved R4 104.2 mm to (27.4, 72.3), turned to 0 degrees
- moved R5 92.1 mm to (27.4, 60.2), turned to 0 degrees
- moved R3 90.1 mm to (40.7, 64.3), turned to 0 degrees
- moved R1 87.3 mm to (27.4, 64.2), turned to 0 degrees
- moved R7 86.7 mm to (40.7, 68.3), turned to 0 degrees
- moved J3 85.5 mm to (77.8, 37.9), turned to 0 degrees
- moved R2 82.7 mm to (27.4, 68.3), turned to 0 degrees
- moved R10 75.9 mm to (70.2, 46.5), turned to 0 degrees
- moved R9 75.3 mm to (58.6, 61.9), turned to 0 degrees
- moved R8 74.6 mm to (70.2, 42.5), turned to 0 degrees
- moved C6 72.6 mm to (70.6, 57.8), turned to 0 degrees
- moved X1 71.7 mm to (48.8, 36.9), turned to 0 degrees
- moved C5 71.7 mm to (75.4, 51.8)
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Routing:
- net +5V: track 198.7 -> 0.00 mm, vias 6 -> 0
- net /CLK8: track 116.5 -> 0.00 mm, vias 4 -> 0
- net /YM_LEFT: track 79.1 -> 0.00 mm, vias 2 -> 0
- net Net-(R4-Pad1): track 76.6 -> 0.00 mm, vias 2 -> 0
- net /D7: track 74.4 -> 0.00 mm
- net /~PSG_CE: track 73.9 -> 0.00 mm
- net /D5: track 73.9 -> 0.00 mm
- net /PSG_OUT: track 73.8 -> 0.00 mm, vias 4 -> 0
- net /D6: track 70.5 -> 0.00 mm
- net /~PSG_WE: track 69.1 -> 0.00 mm
- net /YM_RIGHT: track 64.7 -> 0.00 mm, vias 2 -> 0
- net /D4: track 54.2 -> 0.00 mm, vias 2 -> 0
- net /CLK4: track 52.9 -> 0.00 mm, vias 2 -> 0
- net /D3: track 47.7 -> 0.00 mm, vias 2 -> 0
- net /D1: track 46.8 -> 0.00 mm, vias 2 -> 0
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- removed copper zone on B.Cu, net GND
Other:
- board size 90.2 x 54.6 mm -> 86.4 x 48.3 mm
- board text removed: "YM2612 & SN76489"
